File: DoubleCam.sch (KiCad schematic (older format))
At the start: 22 parts, among them J1 Conn_01x24_MountingPin, J2 Conn_01x24_MountingPin, J3 Conn_02x20_Odd_Even, U1 XC6206PxxxMR, U2 XC6206PxxxMR, X1 SG-3225CAN

Commit message: changed FPC connect
Parts:
- U1, U2: footprint Package_TO_SOT_SMD:SOT-23 -> Package_TO_SOT_SMD:SOT-89-3
- X1: symbol Oscillator:SG-3225CAN -> DoubleCam-rescue:SG-3225CAN-Oscillator
Connections:
- net +1V5: now also J1.15 (Pin_15), J2.15 (Pin_15); no longer J1.10 (Pin_10), J2.10 (Pin_10)
- net +2V8: now also J1.14 (Pin_14), J1.2 (Pin_2), J1.21 (Pin_21), J2.14 (Pin_14), J2.2 (Pin_2), J2.21 (Pin_21); no longer J1.11 (Pin_11), J1.4 (Pin_4), J2.11 (Pin_11), J2.4 (Pin_4)
- net GND: now also J1.1 (Pin_1), J1.10 (Pin_10), J1.23 (Pin_23), J2.1 (Pin_1), J2.10 (Pin_10), J2.23 (Pin_23); no longer J1.15 (Pin_15), J1.2 (Pin_2), J2.15 (Pin_15), J2.2 (Pin_2), J3.1 (Pin_1)
- net OV1_D0: now also J1.6 (Pin_6), J3.6 (Pin_6); no longer J1.19 (Pin_19), J3.15 (Pin_15)
- net OV1_D1: now also J1.4 (Pin_4), J3.4 (Pin_4); no longer J1.21 (Pin_21), J3.17 (Pin_17)
- net OV1_D2: now also J1.3 (Pin_3), J3.3 (Pin_3); no longer J1.22 (Pin_22), J3.18 (Pin_18)
- net OV1_D3: now also J1.5 (Pin_5), J3.5 (Pin_5); no longer J1.20 (Pin_20), J3.16 (Pin_16)
- net OV1_D4: now also J1.7 (Pin_7), J3.7 (Pin_7); no longer J1.18 (Pin_18), J3.14 (Pin_14)
- net OV1_D5: now also J1.9 (Pin_9), J3.9 (Pin_9); no longer J1.16 (Pin_16), J3.12 (Pin_12)
- net OV1_D6: now also J1.11 (Pin_11), J3.10 (Pin_10); no longer J1.14 (Pin_14), J3.11 (Pin_11)
- net OV1_D7: now also J1.13 (Pin_13), J3.12 (Pin_12); no longer J1.12 (Pin_12), J3.9 (Pin_9)
- net OV1_HREF: now also J1.16 (Pin_16), J3.13 (Pin_13); no longer J1.9 (Pin_9), J3.8 (Pin_8)
- net OV1_PCLK: now also J1.8 (Pin_8), J3.8 (Pin_8); no longer J1.17 (Pin_17), J3.13 (Pin_13)
- net OV1_PWDN: now also J1.17 (Pin_17), J3.14 (Pin_14); no longer J1.8 (Pin_8), J3.7 (Pin_7)
- net OV1_RESET: now also J1.19 (Pin_19), J3.16 (Pin_16); no longer J1.6 (Pin_6), J3.5 (Pin_5)
- net OV1_SCL: now also J1.20 (Pin_20), J3.17 (Pin_17); no longer J1.5 (Pin_5), J3.4 (Pin_4)
- net OV1_SDA: now also J1.22 (Pin_22), J3.18 (Pin_18); no longer J1.3 (Pin_3), J3.3 (Pin_3)
- net OV1_VSYNC: now also J1.18 (Pin_18), J3.15 (Pin_15); no longer J1.7 (Pin_7), J3.6 (Pin_6)
- net OV1_XCLK: now also J1.12 (Pin_12), J3.11 (Pin_11); no longer J1.13 (Pin_13), J3.10 (Pin_10)
- net OV2_D0: now also J2.6 (Pin_6), J3.23 (Pin_23); no longer J2.19 (Pin_19), J3.34 (Pin_34)
- net OV2_D1: now also J2.4 (Pin_4), J3.21 (Pin_21); no longer J2.21 (Pin_21), J3.36 (Pin_36)
- net OV2_D2: now also J2.3 (Pin_3), J3.22 (Pin_22); no longer J2.22 (Pin_22), J3.35 (Pin_35)
- net OV2_D3: now also J2.5 (Pin_5), J3.24 (Pin_24); no longer J2.20 (Pin_20), J3.33 (Pin_33)
- net OV2_D4: now also J2.7 (Pin_7), J3.26 (Pin_26); no longer J2.18 (Pin_18), J3.31 (Pin_31)
- net OV2_D5: now also J2.9 (Pin_9), J3.28 (Pin_28); no longer J2.16 (Pin_16), J3.29 (Pin_29)
- net OV2_D6: now also J2.11 (Pin_11), J3.27 (Pin_27); no longer J2.14 (Pin_14), J3.30 (Pin_30)
- net OV2_D7: now also J2.13 (Pin_13), J3.29 (Pin_29); no longer J2.12 (Pin_12), J3.28 (Pin_28)
- net OV2_HREF: now also J2.16 (Pin_16), J3.32 (Pin_32); no longer J2.9 (Pin_9), J3.25 (Pin_25)
- net OV2_PCLK: now also J2.8 (Pin_8), J3.25 (Pin_25); no longer J2.17 (Pin_17), J3.32 (Pin_32)
- net OV2_PWDN: now also J2.17 (Pin_17), J3.31 (Pin_31); no longer J2.8 (Pin_8), J3.26 (Pin_26)
- net OV2_RESET: now also J2.19 (Pin_19), J3.33 (Pin_33); no longer J2.6 (Pin_6), J3.24 (Pin_24)
- net OV2_SCL: now also J2.20 (Pin_20), J3.36 (Pin_36); no longer J2.5 (Pin_5), J3.21 (Pin_21)
- net OV2_SDA: now also J2.22 (Pin_22), J3.35 (Pin_35); no longer J2.3 (Pin_3), J3.22 (Pin_22)
- net OV2_VSYNC: now also J2.18 (Pin_18), J3.34 (Pin_34); no longer J2.7 (Pin_7), J3.23 (Pin_23)
- net OV2_XCLK: now also J2.12 (Pin_12), J3.30 (Pin_30); no longer J2.13 (Pin_13), J3.27 (Pin_27)
- net +5V: no longer names the net of J3.2 (Pin_2)
- no-connect marks 6 -> 4
Other:
- moved on the sheet: J1, J2
